File: receptoresp.kicad_pcb (KiCad board)
At the start: 2 copper layers, 48 x 59 mm, 6 parts

Commit message: capacitor colocado para o modulo nrf
Parts:
- added C1: C, Capacitor_THT:C_Disc_D3.0mm_W1.6mm_P2.50mm, F.Cu at (153.5, 99.5)
- moved NR1 0.71 mm to (173.8, 102.8)
Connections:
- NR1 pad 2: Net-(E1-3V3) -> Net-(NR1-VCC)
Routing:
- net Net-(E1-3V3): track 7.52 -> 2.71 mm
- net Net-(NR1-VCC): track 0.00 -> 4.28 mm
- net Net-(NR1-GND): track 36.1 -> 37.3 mm
- net Net-(E1-D22): track 60.4 -> 59.5 mm
- net Net-(E1-D23): track 47.4 -> 46.7 mm
- net Net-(E1-D19): track 36.5 -> 37.1 mm
- net Net-(E1-D5): track 27.2 -> 26.7 mm
