File: receptoresp.kicad_pcb (KiCad board)
At the start: 2 copper layers, 48 x 59 mm, 7 parts

Commit message: pcb pi pico
Parts:
- removed ? (x3): , 
- removed C1: C_Polarized, Capacitor_THT:C_Disc_D3.0mm_W1.6mm_P2.50mm
- removed E1: ESP-WROOM-32, ESPF:ESP-WROOM-32
- removed REF**: MountingHole_2.2mm_M2_ISO7380, MountingHole:MountingHole_2.2mm_M2_ISO7380
- added A1: RaspberryPi_Pico, Module:RaspberryPi_Pico_Common_THT, F.Cu at (83.0, 57.0)
- added C100uF1: C_Polarized, Capacitor_THT:C_Radial_D4.0mm_H5.0mm_P1.50mm, F.Cu at (102.0, 112.5)
- NR1: footprint nrf:NRF24L01 -> RF_Module:nRF24L01_Breakout
- moved NR1 77.5 mm to (96.6, 110.5), turned to -90 degrees
Connections:
- NR1 pad 8: Net-(E1-D5) -> unconnected-(NR1-IRQ-Pad8)
Routing:
- net Net-(A1-GPIO5): track 10.5 -> 60.8 mm
- net Net-(A1-3V3): track 10.7 -> 56.2 mm
- net Net-(E1-D5): track 26.7 -> 0.00 mm
- net Net-(NR1-GND): track 37.3 -> 17.7 mm
- net Net-(A1-GPIO3): track 46.7 -> 55.6 mm
- net Net-(A1-GPIO4): track 37.1 -> 43.7 mm
- net Net-(A1-GPIO2): track 55.1 -> 50.9 mm
- net Net-(A1-GPIO0): track 59.5 -> 58.0 mm
- removed copper zone on B.Cu, net (none)
Other:
- board size 48 x 59 mm -> 28 x 66 mm

Commit message: one face
Connections:
- A1 pad 10: unconnected-(A1-GPIO7-Pad10) -> Net-(A1-GPIO7)
- A1 pad 5: Net-(A1-GPIO3) -> unconnected-(A1-GPIO3-Pad5)
- NR1 pad 6: Net-(A1-GPIO3) -> Net-(A1-GPIO7)
Routing:
- net Net-(A1-GPIO3): track 55.6 -> 0.00 mm
- net Net-(A1-GPIO7): track 0.00 -> 42.9 mm
- net Net-(A1-GPIO5): track 60.8 -> 62.5 mm
Changed lines of the file:
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@@
 			(layers "*.Cu" "*.Mask")
 			(remove_unused_layers no)
-			(net "Net-(A1-GPIO3)")
+			(net "unconnected-(A1-GPIO3-Pad5)")
 			(pinfunction "GPIO3_5")
 			(pintype "bidirectional")
@@
 			(layers "*.Cu" "*.Mask")
 			(remove_unused_layers no)
-			(net "unconnected-(A1-GPIO7-Pad10)")
+			(net "Net-(A1-GPIO7)")
 			(pinfunction "GPIO7_10")
 			(pintype "bidirectional")
@@
 			(layers "*.Cu" "*.Mask")
 			(remove_unused_layers no)
-			(net "Net-(A1-GPIO3)")
+			(net "Net-(A1-GPIO7)")
 			(pinfunction "MOSI_6")
 			(pintype "input")
@@
 	)
 	(segment
+		(start 94.08 110.46)
+		(end 94.08 68.08)
+		(width 1.5)
+		(layer "B.Cu")
+		(net "Net-(A1-GPIO0)")
+	)
+	(segment
+		(start 94.08 68.08)
+		(end 83 57)
+		(width 1.5)
+		(layer "B.Cu")
+		(net "Net-(A1-GPIO0)")
+	)
+	(segment
 		(start 101.61 110.46)
 		(end 101.61 110.39)
-		(width 1.2)
+		(width 1.5)
 		(layer "B.Cu")
 		(net "Net-(NR1-GND)")
@@
 		(start 101.61 110.46)
 		(end 102 110.85)
-		(width 1.2)
+		(width 1.5)
 		(layer "B.Cu")
 		(net "Net-(NR1-GND)")
@@
 		(start 103 109)
 		(end 103 101.7)
-		(width 1.2)
+		(width 1.5)
 		(layer "B.Cu")
 		(net "Net-(NR1-GND)")
@@
 		(start 101.48 100.18)
 		(end 100.78 100.18)
-		(width 1.2)
+		(width 1.5)
 		(layer "B.Cu")
 		(net "Net-(NR1-GND)")
@@
 		(start 96.62 110.46)
 		(end 101.61 110.46)
-		(width 1.2)
+		(width 1.5)
 		(layer "B.Cu")
 		(net "Net-(NR1-GND)")
@@
 		(start 103 101.7)
 		(end 101.48 100.18)
-		(width 1.2)
+		(width 1.5)
 		(layer "B.Cu")
 		(net "Net-(NR1-GND)")
@@
 		(start 101.61 110.39)
 		(end 103 109)
-		(width 1.2)
+		(width 1.5)
 		(layer "B.Cu")
 		(net "Net-(NR1-GND)")
+	)
+	(segment
+		(start 91.54 70.54)
+		(end 91.54 110.46)
+		(width 1.5)
+		(layer "B.Cu")
+		(net "Net-(A1-GPIO2)")
+	)
+	(segment
+		(start 85.62 64.62)
+		(end 91.54 70.54)
+		(width 1.5)
+		(layer "B.Cu")
+		(net "Net-(A1-GPIO2)")
+	)
+	(segment
+		(start 83 64.62)
+		(end 85.62 64.62)
+		(width 1.5)
+		(layer "B.Cu")
+		(net "Net-(A1-GPIO2)")
+	)
+	(segment
+		(start 89 110.46)
+		(end 89 75.7)
+		(width 1.5)
+		(layer "B.Cu")
+		(net "Net-(A1-GPIO4)")
+	)
+	(segment
+		(start 89 75.7)
+		(end 83 69.7)
+		(width 1.5)
+		(layer "B.Cu")
+		(net "Net-(A1-GPIO4)")
 	)
 	(segment
 		(start 96.62 113)
 		(end 101.55 113)
-		(width 1.2)
+		(width 1.5)
 		(layer "B.Cu")
 		(net "Net-(A1-3V3)")
@@
 		(start 105 69)
 		(end 103.16 67.16)
-		(width 1.2)
+		(width 1.5)
 		(layer "B.Cu")
 		(net "Net-(A1-3V3)")
@@
 		(start 101.55 113)
 		(end 102 113)
-		(width 1.2)
+		(width 1.5)
 		(layer "B.Cu")
 		(net "Net-(A1-3V3)")
@@
 		(start 101.55 113)
 		(end 102 112.55)
-		(width 1.2)
+		(width 1.5)
 		(layer "B.Cu")
 		(net "Net-(A1-3V3)")
@@
 		(start 103.16 67.16)
 		(end 100.78 67.16)
-		(width 1.2)
+		(width 1.5)
 		(layer "B.Cu")
 		(net "Net-(A1-3V3)")
@@
 		(start 102 113)
 		(end 105 110)
-		(width 1.2)
+		(width 1.5)
 		(layer "B.Cu")
 		(net "Net-(A1-3V3)")
@@
 		(start 105 110)
 		(end 105 69)
-		(width 1.2)
+		(width 1.5)
 		(layer "B.Cu")
 		(net "Net-(A1-3V3)")
+	)
+	(segment
+		(start 87 115)
+		(end 86 114)
+		(width 1.5)
+		(layer "B.Cu")
+		(net "Net-(A1-GPIO7)")
+	)
+	(segment
+		(start 90.742081 115)
+		(end 87 115)
+		(width 1.5)
+		(layer "B.Cu")
+		(net "Net-(A1-GPIO7)")
+	)
+	(segment
+		(start 91.54 113)
+		(end 91.54 114.202081)
+		(width 1.5)
+		(layer "B.Cu")
+		(net "Net-(A1-GPIO7)")
+	)
+	(segment
+		(start 91.54 114.202081)
+		(end 90.742081 115)
+		(width 1.5)
+		(layer "B.Cu")
+		(net "Net-(A1-GPIO7)")
+	)
+	(segment
+		(start 86 114)
+		(end 86 82.86)
+		(width 1.5)
+		(layer "B.Cu")
+		(net "Net-(A1-GPIO7)")
+	)
+	(segment
+		(start 86 82.86)
+		(end 83 79.86)
+		(width 1.5)
+		(layer "B.Cu")
+		(net "Net-(A1-GPIO7)")
+	)
+	(segment
+		(start 92.25 117.75)
+		(end 85.75 117.75)
+		(width 1.5)
+		(layer "B.Cu")
+		(net "Net-(A1-GPIO5)")
 	)
 	(segment
 		(start 80 73)
 		(end 80.76 72.24)
-		(width 1.2)
+		(width 1.5)
+		(layer "B.Cu")
+		(net "Net-(A1-GPIO5)")
+	)
+	(segment
+		(start 94.08 115.92)
+		(end 92.25 117.75)
+		(width 1.5)
+		(layer "B.Cu")
+		(net "Net-(A1-GPIO5)")
+	)
+	(segment
+		(start 94.08 113)
+		(end 94.08 115.92)
+		(width 1.5)
+		(layer "B.Cu")
+		(net "Net-(A1-GPIO5)")
+	)
+	(segment
+		(start 85.75 117.75)
+		(end 80 112)
+		(width 1.5)
 		(layer "B.Cu")
 		(net "Net-(A1-GPIO5)")
@@
 		(start 80.76 72.24)
 		(end 83 72.24)
-		(width 1.2)
+		(width 1.5)
 		(layer "B.Cu")
 		(net "Net-(A1-GPIO5)")
@@
 		(start 80 112)
 		(end 80 73)
-		(width 1.2)
+		(width 1.5)
 		(layer "B.Cu")
 		(net "Net-(A1-GPIO5)")
 	)
-	(segment
-		(start 91.282081 117)
-		(end 85 117)
-		(width 1.2)
-		(layer "B.Cu")
-		(net "Net-(A1-GPIO5)")
-	)
-	(segment
-		(start 94.08 113)
-		(end 94.08 114.202081)
-		(width 1.2)
-		(layer "B.Cu")
-		(net "Net-(A1-GPIO5)")
-	)
-	(segment
-		(start 85 117)
-		(end 80 112)
-		(width 1.2)
-		(layer "B.Cu")
-		(net "Net-(A1-GPIO5)")
-	)
-	(segment
-		(start 94.08 114.202081)
-		(end 91.282081 117)
-		(width 1.2)
-		(layer "B.Cu")
-		(net "Net-(A1-GPIO5)")
-	)
-	(segment
-		(start 88 74)
-		(end 83.7 69.7)
-		(width 1.2)
-		(layer "F.Cu")
-		(net "Net-(A1-GPIO4)")
-	)
-	(segment
-		(start 89 110.46)
-		(end 88 109.46)
-		(width 1.2)
-		(layer "F.Cu")
-		(net "Net-(A1-GPIO4)")
-	)
-	(segment
-		(start 83.7 69.7)
-		(end 83 69.7)
-		(width 1.2)
-		(layer "F.Cu")
-		(net "Net-(A1-GPIO4)")
-	)
-	(segment
-		(start 88 109.46)
-		(end 88 74)
-		(width 1.2)
-		(layer "F.Cu")
-		(net "Net-(A1-GPIO4)")
-	)
-	(segment
-		(start 94.08 110.46)
-		(end 94.08 68.08)
-		(width 1.2)
-		(layer "B.Cu")
-		(net "Net-(A1-GPIO0)")
-	)
-	(segment
-		(start 94.08 68.08)
-		(end 83 57)
-		(width 1.2)
-		(layer "B.Cu")
-		(net "Net-(A1-GPIO0)")
-	)
-	(segment
-		(start 90.742081 115)
-		(end 87 115)
-		(width 1.2)
-		(layer "B.Cu")
-		(net "Net-(A1-GPIO3)")
-	)
-	(segment
-		(start 87 115)
-		(end 86 114)
-		(width 1.2)
-		(layer "B.Cu")
-		(net "Net-(A1-GPIO3)")
-	)
-	(segment
-		(start 86 70.16)
-		(end 83 67.16)
-		(width 1.2)
-		(layer "B.Cu")
-		(net "Net-(A1-GPIO3)")
-	)
-	(segment
-		(start 91.54 113)
-		(end 91.54 114.202081)
-		(width 1.2)
-		(layer "B.Cu")
-		(net "Net-(A1-GPIO3)")
-	)
-	(segment
-		(start 91.54 114.202081)
-		(end 90.742081 115)
-		(width 1.2)
-		(layer "B.Cu")
-		(net "Net-(A1-GPIO3)")
-	)
-	(segment
-		(start 86 114)
-		(end 86 70.16)
-		(width 1.2)
-		(layer "B.Cu")
-		(net "Net-(A1-GPIO3)")
-	)
-	(segment
-		(start 91.54 70.54)
-		(end 91.54 110.46)
-		(width 1.2)
-		(layer "B.Cu")
-		(net "Net-(A1-GPIO2)")
-	)
-	(segment
-		(start 85.62 64.62)
-		(end 91.54 70.54)
-		(width 1.2)
-		(layer "B.Cu")
-		(net "Net-(A1-GPIO2)")
-	)
-	(segment
-		(start 83 64.62)
-		(end 85.62 64.62)
-		(width 1.2)
-		(layer "B.Cu")
-		(net "Net-(A1-GPIO2)")
-	)
-	(zone
-		(layers "F.Cu" "B.Cu" "Edge.Cuts")
-		(name "a")
-		(hatch edge 0.5)
-		(connect_pads
-			(clearance 0)
-		)
-		(min_thickness 0.3)
-		(keepout
-			(tracks not_allowed)
-			(vias not_allowed)
-			(pads not_allowed)
-			(copperpour not_allowed)
-			(footprints not_allowed)
-		)
-		(placement
-			(enabled no)
-			(sheetname "/")
-		)
-		(fill
-			(thermal_gap 0.7)
-			(thermal_bridge_width 0.7)
-			(island_removal_mode 1)
-		)
-		(polygon
-			(pts
-				(xy 78 53) (xy 106 53) (xy 106 119) (xy 78 119)
-			)
-		)
-	)
 	(embedded_fonts no)
