File: _restore_backup_2026-05-15T14-30-06-863/receptoresp.kicad_sch (KiCad schematic)
At the start: 3 parts

Commit message: capacitor polalizado 100uF
Parts:
- C1: footprint Capacitor_THT:C_Disc_D3.0mm_W1.6mm_P2.50mm -> (none)
Changed lines of the file:
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@@
 			)
 		)
-		(property "Footprint" "Capacitor_THT:C_Disc_D3.0mm_W1.6mm_P2.50mm"
+		(property "Footprint" ""
 			(at 180.0352 101.6 0)
 			(hide yes)
